Commit message: update

File: DtachableHead_urdf/urdf/DtachableHead_urdf.urdf (robot description, URDF)
Before this commit: robot DtachableHead_urdf, 7 links, 6 joints
Links:
- link link4: mass 0.0459058932133953 -> 0.0459058932133952
- link link5: mass 0.0531974022503482 -> 0.0531974022503484
Joints:
- joint Joint2: origin xyz=-0.0400000000000002 0 -0.0390000000000001 rpy=0 1.5707963267949 0 -> xyz=-0.04 0 -0.039 rpy=0 1.5708 0
- joint Joint5: origin xyz=0.0209400000000001 0 0.0414999999999974 rpy=1.5707963267949 0 1.5707963267949 -> xyz=0.02094 0 0.0415 rpy=1.5708 0 1.5708
- joint Joint6: origin xyz=0.0209399999999999 0.0675000000000001 -0.0210000000000012 rpy=0 -1.5707963267949 0 -> xyz=0.0209399999999999 0.0675000000000001 -0.0210000000000012 rpy=0 1.5707963267949 0
