Commit message: update

File: DtachableHead_L515_urdf/urdf/DtachableHead_L515_urdf.urdf (robot description, URDF)
Before this commit: robot DtachableHead_L515_urdf, 8 links, 7 joints
Joints:
- joint joint7: origin xyz=-0.00010025 -0.0089999 -0.029479 rpy=1.5708 1.5708 0 -> xyz=-0.00010025 -0.0089999 -0.029479 rpy=0 0 0
